Commit message: The multiple trajectory visualization with shaded regions and comparisons between CRCLF and regular CLF

File: src/daadbot_desc/urdf/2_link_urdf/2link_robot_fixed.urdf (robot description, URDF)
Before this commit: robot 2link_robot, 5 links, 4 joints
Joints:
- joint baseHinge: limit lower=-1000.0 upper=1000.0 effort=50.0 velocity=1.0 -> lower=-1000.0 upper=1000.0 effort=50.0 velocity=0.5
- joint interArm: limit lower=-1000.0 upper=1000.0 effort=30.0 velocity=1.0 -> lower=-1000.0 upper=1000.0 effort=30.0 velocity=0.5

File: src/daadbot_desc/urdf/2_link_urdf/2link_robot_fixed.urdf.xacro (robot description, xacro)
@@ -46,5 +46,5 @@
     <joint name="baseHinge" type="revolute">
         <axis rpy="0 0 0" xyz="0 0 1" />
-        <limit effort="50.0" velocity="1.0" lower="-1000.0" upper="1000.0" />
+        <limit effort="50.0" velocity="0.5" lower="-1000.0" upper="1000.0" />
         <parent link="base" />
         <child link="arm1" />
@@ -72,5 +72,5 @@
     <joint name="interArm" type="revolute">
         <axis rpy="0 0 0" xyz="0 0 1" />
-        <limit effort="30.0" velocity="1.0" lower="-1000.0" upper="1000.0" />
+        <limit effort="30.0" velocity="0.5" lower="-1000.0" upper="1000.0" />
         <parent link="arm1" />
         <child link="arm2" />
