Commit message: lower dof versions of a urdf with full controller, configs, and bringup ctc controller for effort command version - lab table

File: daadbot_desc/urdf/urdf_table_pos_j6m90_2dof/daadbot.urdf (robot description, URDF)
Before this commit: robot daadbot, 29 links, 28 joints
Joints:
- joint base_claw_joint1: axis 0 0 -1 -> (none); limit lower=0 upper=0.9 effort=5 velocity=10 -> (none); mimic joint=gear1_joint multiplier=-1 offset=0 -> (none); type revolute -> fixed
- joint base_claw_joint2: axis 0 0 1 -> (none); limit lower=0 upper=0.9 effort=5 velocity=10 -> (none); mimic joint=gear1_joint multiplier=-1 offset=0 -> (none); type revolute -> fixed
- joint claw_joint1: axis 0 0 1 -> (none); limit lower=0 upper=0.9 effort=5 velocity=10 -> (none); mimic joint=base_claw_joint1 multiplier=1 offset=0 -> (none); type revolute -> fixed
- joint claw_joint2: axis 0 0 1 -> (none); limit lower=-0.9 upper=0 effort=5 velocity=10 -> (none); mimic joint=base_claw_joint2 multiplier=-1 offset=0 -> (none); type revolute -> fixed
- joint gear1_joint: axis 0 0 -1 -> (none); limit lower=-0.9 upper=0 effort=5 velocity=10 -> (none); type revolute -> fixed
- joint gear2_joint: axis 0 0 -1 -> (none); limit lower=-0.9 upper=0.9 effort=5 velocity=10 -> (none); mimic joint=gear1_joint multiplier=-1 offset=0 -> (none); type revolute -> fixed
- joint joint_3: axis 0 0 -1 -> (none); limit lower=-0.1 upper=3.2 effort=200.0 velocity=12.776 -> (none); type revolute -> fixed
- joint joint_4: axis 0 0 -1 -> (none); limit lower=-1.9199 upper=1.9199 effort=200.0 velocity=12.77581 -> (none); type revolute -> fixed
- joint joint_5: axis 0 0 -1 -> (none); limit lower=-0.785398 upper=0.785398 effort=15 velocity=6.0 -> (none); type revolute -> fixed
- joint joint_6: axis 0 0 -1 -> (none); limit lower=-0.785398 upper=0.785398 effort=15 velocity=6.0 -> (none); type revolute -> fixed
- joint joint_7: axis 0 0 -1 -> (none); limit lower=-0.785398 upper=0.785398 effort=15 velocity=6.0 -> (none); type revolute -> fixed

File: daadbot_desc/urdf/urdf_table_pos_j6m90_3dof/daadbot.urdf (robot description, URDF)
Before this commit: robot daadbot, 29 links, 28 joints
Joints:
- joint base_claw_joint1: axis 0 0 -1 -> (none); limit lower=0 upper=0.9 effort=5 velocity=10 -> (none); mimic joint=gear1_joint multiplier=-1 offset=0 -> (none); type revolute -> fixed
- joint base_claw_joint2: axis 0 0 1 -> (none); limit lower=0 upper=0.9 effort=5 velocity=10 -> (none); mimic joint=gear1_joint multiplier=-1 offset=0 -> (none); type revolute -> fixed
- joint claw_joint1: axis 0 0 1 -> (none); limit lower=0 upper=0.9 effort=5 velocity=10 -> (none); mimic joint=base_claw_joint1 multiplier=1 offset=0 -> (none); type revolute -> fixed
- joint claw_joint2: axis 0 0 1 -> (none); limit lower=-0.9 upper=0 effort=5 velocity=10 -> (none); mimic joint=base_claw_joint2 multiplier=-1 offset=0 -> (none); type revolute -> fixed
- joint gear1_joint: axis 0 0 -1 -> (none); limit lower=-0.9 upper=0 effort=5 velocity=10 -> (none); type revolute -> fixed
- joint gear2_joint: axis 0 0 -1 -> (none); limit lower=-0.9 upper=0.9 effort=5 velocity=10 -> (none); mimic joint=gear1_joint multiplier=-1 offset=0 -> (none); type revolute -> fixed
- joint joint_4: axis 0 0 -1 -> (none); limit lower=-1.9199 upper=1.9199 effort=200.0 velocity=12.77581 -> (none); type revolute -> fixed
- joint joint_5: axis 0 0 -1 -> (none); limit lower=-0.785398 upper=0.785398 effort=15 velocity=6.0 -> (none); type revolute -> fixed
- joint joint_6: axis 0 0 -1 -> (none); limit lower=-0.785398 upper=0.785398 effort=15 velocity=6.0 -> (none); type revolute -> fixed
- joint joint_7: axis 0 0 -1 -> (none); limit lower=-0.785398 upper=0.785398 effort=15 velocity=6.0 -> (none); type revolute -> fixed

File: daadbot_desc/urdf/urdf_table_pos_j6m90_4dof/daadbot.urdf (robot description, URDF)
Before this commit: robot daadbot, 29 links, 28 joints
Joints:
- joint base_claw_joint1: axis 0 0 -1 -> (none); limit lower=0 upper=0.9 effort=5 velocity=10 -> (none); mimic joint=gear1_joint multiplier=-1 offset=0 -> (none); type revolute -> fixed
- joint base_claw_joint2: axis 0 0 1 -> (none); limit lower=0 upper=0.9 effort=5 velocity=10 -> (none); mimic joint=gear1_joint multiplier=-1 offset=0 -> (none); type revolute -> fixed
- joint claw_joint1: axis 0 0 1 -> (none); limit lower=0 upper=0.9 effort=5 velocity=10 -> (none); mimic joint=base_claw_joint1 multiplier=1 offset=0 -> (none); type revolute -> fixed
- joint claw_joint2: axis 0 0 1 -> (none); limit lower=-0.9 upper=0 effort=5 velocity=10 -> (none); mimic joint=base_claw_joint2 multiplier=-1 offset=0 -> (none); type revolute -> fixed
- joint gear1_joint: axis 0 0 -1 -> (none); limit lower=-0.9 upper=0 effort=5 velocity=10 -> (none); type revolute -> fixed
- joint gear2_joint: axis 0 0 -1 -> (none); limit lower=-0.9 upper=0.9 effort=5 velocity=10 -> (none); mimic joint=gear1_joint multiplier=-1 offset=0 -> (none); type revolute -> fixed
- joint joint_5: axis 0 0 -1 -> (none); limit lower=-0.785398 upper=0.785398 effort=15 velocity=6.0 -> (none); type revolute -> fixed
- joint joint_6: axis 0 0 -1 -> (none); limit lower=-0.785398 upper=0.785398 effort=15 velocity=6.0 -> (none); type revolute -> fixed
- joint joint_7: axis 0 0 -1 -> (none); limit lower=-0.785398 upper=0.785398 effort=15 velocity=6.0 -> (none); type revolute -> fixed

File: daadbot_desc/urdf/urdf_table_pos_j6m90_5dof/daadbot.urdf (robot description, URDF)
Before this commit: robot daadbot, 29 links, 28 joints
Joints:
- joint base_claw_joint1: axis 0 0 -1 -> (none); limit lower=0 upper=0.9 effort=5 velocity=10 -> (none); mimic joint=gear1_joint multiplier=-1 offset=0 -> (none); type revolute -> fixed
- joint base_claw_joint2: axis 0 0 1 -> (none); limit lower=0 upper=0.9 effort=5 velocity=10 -> (none); mimic joint=gear1_joint multiplier=-1 offset=0 -> (none); type revolute -> fixed
- joint claw_joint1: axis 0 0 1 -> (none); limit lower=0 upper=0.9 effort=5 velocity=10 -> (none); mimic joint=base_claw_joint1 multiplier=1 offset=0 -> (none); type revolute -> fixed
- joint claw_joint2: axis 0 0 1 -> (none); limit lower=-0.9 upper=0 effort=5 velocity=10 -> (none); mimic joint=base_claw_joint2 multiplier=-1 offset=0 -> (none); type revolute -> fixed
- joint gear1_joint: axis 0 0 -1 -> (none); limit lower=-0.9 upper=0 effort=5 velocity=10 -> (none); type revolute -> fixed
- joint gear2_joint: axis 0 0 -1 -> (none); limit lower=-0.9 upper=0.9 effort=5 velocity=10 -> (none); mimic joint=gear1_joint multiplier=-1 offset=0 -> (none); type revolute -> fixed
- joint joint_5: limit lower=-0.785398 upper=0.785398 effort=15 velocity=6.0 -> lower=-0.1 upper=3.4 effort=15 velocity=19.896753
- joint joint_6: axis 0 0 -1 -> (none); limit lower=-0.785398 upper=0.785398 effort=15 velocity=6.0 -> (none); type revolute -> fixed
- joint joint_7: axis 0 0 -1 -> (none); limit lower=-0.785398 upper=0.785398 effort=15 velocity=6.0 -> (none); type revolute -> fixed

File: daadbot_desc/urdf/urdf_table_pos_j6m90_6dof/daadbot.urdf (robot description, URDF)
Before this commit: robot daadbot, 29 links, 28 joints
Joints:
- joint base_claw_joint1: axis 0 0 -1 -> (none); limit lower=0 upper=0.9 effort=5 velocity=10 -> (none); mimic joint=gear1_joint multiplier=-1 offset=0 -> (none); type revolute -> fixed
- joint base_claw_joint2: axis 0 0 1 -> (none); limit lower=0 upper=0.9 effort=5 velocity=10 -> (none); mimic joint=gear1_joint multiplier=-1 offset=0 -> (none); type revolute -> fixed
- joint claw_joint1: axis 0 0 1 -> (none); limit lower=0 upper=0.9 effort=5 velocity=10 -> (none); mimic joint=base_claw_joint1 multiplier=1 offset=0 -> (none); type revolute -> fixed
- joint claw_joint2: axis 0 0 1 -> (none); limit lower=-0.9 upper=0 effort=5 velocity=10 -> (none); mimic joint=base_claw_joint2 multiplier=-1 offset=0 -> (none); type revolute -> fixed
- joint gear1_joint: axis 0 0 -1 -> (none); limit lower=-0.9 upper=0 effort=5 velocity=10 -> (none); type revolute -> fixed
- joint gear2_joint: axis 0 0 -1 -> (none); limit lower=-0.9 upper=0.9 effort=5 velocity=10 -> (none); mimic joint=gear1_joint multiplier=-1 offset=0 -> (none); type revolute -> fixed
- joint joint_5: limit lower=-0.785398 upper=0.785398 effort=15 velocity=6.0 -> lower=-0.1 upper=3.4 effort=15 velocity=19.896753
- joint joint_6: limit lower=-0.785398 upper=0.785398 effort=15 velocity=6.0 -> lower=-3.673205e-06 upper=3.141596326795 effort=15 velocity=19.897
- joint joint_7: axis 0 0 -1 -> (none); limit lower=-0.785398 upper=0.785398 effort=15 velocity=6.0 -> (none); type revolute -> fixed
