Commit message: moveit configuration for the selected config lab table urdf

File: daadbot_desc/urdf/urdf_table_pos_j6m90/daadbot.urdf (robot description, URDF)
Before this commit: robot daadbot, 29 links, 28 joints
Joints:
- joint joint_2: limit lower=-3.4907 upper=0.5236 effort=200.0 velocity=12.776 -> lower=-3.307 upper=0.5236 effort=200.0 velocity=12.776

File: daadbot_desc/urdf/urdf_table_pos_j6m90_2dof/daadbot.urdf (robot description, URDF)
Before this commit: robot daadbot, 29 links, 28 joints
Joints:
- joint joint_2: limit lower=-3.4907 upper=0.5236 effort=200.0 velocity=12.776 -> lower=-3.307 upper=0.5236 effort=200.0 velocity=12.776

File: daadbot_desc/urdf/urdf_table_pos_j6m90_2dof_trunc/daadbot.urdf (robot description, URDF)
Before this commit: robot daadbot, 12 links, 11 joints
Joints:
- joint joint_2: limit lower=-3.4907 upper=0.5236 effort=200.0 velocity=12.776 -> lower=-3.307 upper=0.5236 effort=200.0 velocity=12.776

File: daadbot_desc/urdf/urdf_table_pos_j6m90_3dof/daadbot.urdf (robot description, URDF)
Before this commit: robot daadbot, 29 links, 28 joints
Joints:
- joint joint_2: limit lower=-3.4907 upper=0.5236 effort=200.0 velocity=12.776 -> lower=-3.307 upper=0.5236 effort=200.0 velocity=12.776

File: daadbot_desc/urdf/urdf_table_pos_j6m90_3dof_trunc/daadbot.urdf (robot description, URDF)
Before this commit: robot daadbot, 14 links, 13 joints
Joints:
- joint joint_2: limit lower=-3.4907 upper=0.5236 effort=200.0 velocity=12.776 -> lower=-3.307 upper=0.5236 effort=200.0 velocity=12.776

File: daadbot_desc/urdf/urdf_table_pos_j6m90_4dof/daadbot.urdf (robot description, URDF)
Before this commit: robot daadbot, 29 links, 28 joints
Joints:
- joint joint_2: limit lower=-3.4907 upper=0.5236 effort=200.0 velocity=12.776 -> lower=-3.307 upper=0.5236 effort=200.0 velocity=12.776

File: daadbot_desc/urdf/urdf_table_pos_j6m90_4dof_trunc/daadbot.urdf (robot description, URDF)
Before this commit: robot daadbot, 16 links, 15 joints
Joints:
- joint joint_2: limit lower=-3.4907 upper=0.5236 effort=200.0 velocity=12.776 -> lower=-3.307 upper=0.5236 effort=200.0 velocity=12.776

File: daadbot_desc/urdf/urdf_table_pos_j6m90_5dof/daadbot.urdf (robot description, URDF)
Before this commit: robot daadbot, 29 links, 28 joints
Joints:
- joint joint_2: limit lower=-3.4907 upper=0.5236 effort=200.0 velocity=12.776 -> lower=-3.307 upper=0.5236 effort=200.0 velocity=12.776

File: daadbot_desc/urdf/urdf_table_pos_j6m90_5dof_trunc/daadbot.urdf (robot description, URDF)
Before this commit: robot daadbot, 18 links, 17 joints
Joints:
- joint joint_2: limit lower=-3.4907 upper=0.5236 effort=200.0 velocity=12.776 -> lower=-3.307 upper=0.5236 effort=200.0 velocity=12.776

File: daadbot_desc/urdf/urdf_table_pos_j6m90_6dof/daadbot.urdf (robot description, URDF)
Before this commit: robot daadbot, 29 links, 28 joints
Joints:
- joint joint_2: limit lower=-3.4907 upper=0.5236 effort=200.0 velocity=12.776 -> lower=-3.307 upper=0.5236 effort=200.0 velocity=12.776

File: daadbot_desc/urdf/urdf_table_pos_j6m90_6dof_trunc/daadbot.urdf (robot description, URDF)
Before this commit: robot daadbot, 20 links, 19 joints
Joints:
- joint joint_2: limit lower=-3.4907 upper=0.5236 effort=200.0 velocity=12.776 -> lower=-3.307 upper=0.5236 effort=200.0 velocity=12.776
